File: MODULE/POWE/KLD1117/SO223/V33D/src/kicadBoard.kicad_sch (KiCad schematic)
At the start: 2 parts

Commit message: Quickly Adding Everything
Parts:
- added U?: VREG-SO223-X-KLD1117-V33D-VR111722333, oomlout_OOMP_parts:VREG-SO223-X-KLD1117-V33D-VR111722333, symbol oomlout_OOMP_parts:VREG-SO223-X-KLD1117-V33D-VR111722333
Connections:
- net GND: now also U?.1 (GND)
- net VIN: now also U?.3 (VI)
- net VOUT: now also U?.2 (VO)
Other:
- note added: "MODULE-POWE KLD1117-SO223-V33D oom.lt/MP1117"
- note removed: "MODULE-POWE KLD1117-SO23-01 oom.lt/MP1117"
Changed lines of the file:
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@@
     (stroke (width 0) (type default) (color 0 0 0 0))
+  )
+  (polyline (pts (xy 28.575 24.765) (xy 124.46 24.765))
+    (stroke (width 0.5) (type solid) (color 0 0 0 1))
   )
   (wire (pts (xy 89.535 59.69) (xy 89.535 66.04))
@@
     (stroke (width 0) (type default) (color 0 0 0 0))
   )
+  (polyline (pts (xy 124.46 92.075) (xy 124.46 24.765))
+    (stroke (width 0.5) (type solid) (color 0 0 0 1))
+  )
   (wire (pts (xy 55.245 59.69) (xy 61.595 59.69))
     (stroke (width 0) (type default) (color 0 0 0 0))
   )
+  (polyline (pts (xy 28.575 24.765) (xy 28.575 92.075))
+    (stroke (width 0.5) (type solid) (color 0 0 0 1))
+  )
   (wire (pts (xy 61.595 59.69) (xy 67.945 59.69))
     (stroke (width 0) (type default) (color 0 0 0 0))
+  )
+  (polyline (pts (xy 28.575 92.075) (xy 124.46 92.075))
+    (stroke (width 0.5) (type solid) (color 0 0 0 1))
   )
   (wire (pts (xy 75.565 76.2) (xy 61.595 76.2))
@@
     (stroke (width 0) (type default) (color 0 0 0 0))
   )
-  (text "MODULE-POWE\nKLD1117-SO23-01\noom.lt/MP1117" (at 50.165 48.895 0)
+  (text "MODULE-POWE\nKLD1117-SO223-V33D\noom.lt/MP1117" (at 50.165 48.895 0)
     (effects (font (size 3 3) (thickness 0.6) bold) (justify left bottom))
   )
@@
     (pin "2")
   )
+  (symbol (lib_id "oomlout_OOMP_parts:VREG-SO223-X-KLD1117-V33D-VR111722333") (at 75.565 59.69 0) (unit 1)
+    (in_bom yes) (on_board yes) (fields_autoplaced)
+    (property "Reference" "U?" (id 0) (at 75.565 52.07 0))
+    (property "Value" "VREG-SO223-X-KLD1117-V33D-VR111722333" (id 1) (at 75.565 54.61 0)
+      (effects (font (size 0.75 0.75)))
+    )
+    (property "Footprint" "oomlout_OOMP_parts:VREG-SO223-X-KLD1117-V33D-VR111722333" (id 2) (at 75.565 54.61 0)
+      (effects (font (size 1.27 1.27)) hide)
+    )
+    (property "Datasheet" "oom.lt/VR111722333" (id 3) (at 78.105 66.04 0)
+      (effects (font (size 1.27 1.27)) hide)
+    )
+    (pin "1")
+    (pin "2")
+    (pin "3")
+  )
   (sheet_instances
     (path "/" (page "1"))
@@
       (reference "C?") (unit 1) (value "CAPC-0603-X-NF100-V50-C6N100") (footprint "oomlout_OOMP_parts:CAPC-0603-X-NF100-V50-C6N100")
     )
+    (path "/618d52fd-329e-4ad1-a093-879c05cb1d62"
+      (reference "U?") (unit 1) (value "VREG-SO223-X-KLD1117-V33D-VR111722333") (footprint "oomlout_OOMP_parts:VREG-SO223-X-KLD1117-V33D-VR111722333")
+    )
   )
